File: carte_comptage/_autosave-carte_comptage.sch (KiCad schematic (older format))
At the start: 38 parts, among them U3.3V MC33269ST-3.3T3G

Commit message: debut xtal a finir
Parts:
- added Crst? (x2): 0.1µC, Capacitor_SMD:C_1206_3216Metric, symbol Device:C
- added Xtal: 16MHz, symbol Device:Crystal_GND23
- renumbered Cbbs to Cbbs1, Cbss to Cbss1, Cdcr to Cdcr1, Crst to Crst1, Db to Db1, Dpow to Dpow1, Dstatus to Dstatus1, Dusb to Dusb1, F to F1, Jbat to Jbat1, Lb to Lb1, Rbc to Rbc1, RledP to RledP1, Rstatus to Rstatus1, SWD to SWD1, SWrst to SWrst1, U3.3V to U3.3V1, USB to USB1, buck to buck1, swBoot to swBoot1, µc to µc1
Connections:
- net GND: now also Crst?.2, Crst?.2, Xtal.2, Xtal.3
- net UART_RX: now also µc1.13 (PA3); no longer µc1.11 (PA1)
- net UART_TX: now also µc1.12 (PA2); no longer µc1.10 (PA0)
- new net: Crst?.1, Xtal.1
- new net: Crst?.1, Xtal.4
