File: carte_comptage/Shield_LoRa.sch (KiCad schematic (older format))
At the start: 5 parts, among them J1 Conn_01x08, J2 Conn_01x06, J3 Conn_01x08, J4 Conn_01x10

Commit message: debut routage
Connections:
- wire segments 24 -> 21
Other:
- moved on the sheet: LoRa1
Changed lines of the file:
@@
 L Connector_Generic:Conn_02x04_Counter_Clockwise LoRa1
 U 1 1 61424C97
-P 3900 2500
-F 0 "LoRa1" H 3950 2725 50  0000 C CNN
-F 1 "Conn_02x04_Counter_Clockwise" H 3950 2726 50  0001 C CNN
-F 2 "Connector_PinSocket_2.54mm:PinSocket_2x04_P2.54mm_Vertical" H 3900 2500 50  0001 C CNN
-F 3 "~" H 3900 2500 50  0001 C CNN
-	1    3900 2500
+P 4350 2200
+F 0 "LoRa1" H 4400 2425 50  0000 C CNN
+F 1 "Conn_02x04_Counter_Clockwise" H 4400 2426 50  0001 C CNN
+F 2 "Connector_PinSocket_2.54mm:PinSocket_2x04_P2.54mm_Vertical" H 4350 2200 50  0001 C CNN
+F 3 "~" H 4350 2200 50  0001 C CNN
+	1    4350 2200
 	1    0    0    -1
 $EndComp
@@
 L power:GND #PWR0101
 U 1 1 6142571F
-P 3300 2550
-F 0 "#PWR0101" H 3300 2300 50  0001 C CNN
-F 1 "GND" H 3400 2650 50  0000 C CNN
-F 2 "" H 3300 2550 50  0001 C CNN
-F 3 "" H 3300 2550 50  0001 C CNN
-	1    3300 2550
+P 3600 2200
+F 0 "#PWR0101" H 3600 1950 50  0001 C CNN
+F 1 "GND" H 3650 2250 50  0000 C CNN
+F 2 "" H 3600 2200 50  0001 C CNN
+F 3 "" H 3600 2200 50  0001 C CNN
+	1    3600 2200
 	1    0    0    -1
 $EndComp
-Wire Wire Line
-	3300 2550 3300 2500
-Text Label 3500 2600 0    50   ~ 0
+Text Label 5000 2300 2    50   ~ 0
 NRST
-Wire Wire Line
-	3700 2600 3500 2600
 $Comp
 L power:+3.3V #PWR0102
 U 1 1 614263C6
-P 3650 2350
-F 0 "#PWR0102" H 3650 2200 50  0001 C CNN
-F 1 "+3.3V" H 3665 2523 50  0000 C CNN
-F 2 "" H 3650 2350 50  0001 C CNN
-F 3 "" H 3650 2350 50  0001 C CNN
-	1    3650 2350
-	1    0    0    -1
+P 4150 2400
+F 0 "#PWR0102" H 4150 2250 50  0001 C CNN
+F 1 "+3.3V" V 4050 2400 50  0000 C CNN
+F 2 "" H 4150 2400 50  0001 C CNN
+F 3 "" H 4150 2400 50  0001 C CNN
+	1    4150 2400
+	0    -1   -1   0
 $EndComp
-Wire Wire Line
-	3650 2350 3650 2400
-Wire Wire Line
-	3650 2400 3700 2400
-Text Label 4550 2400 2    50   ~ 0
+Text Label 3750 2100 0    50   ~ 0
 SPI_SCK
-Text Label 4550 2500 2    50   ~ 0
+Text Label 3750 2300 0    50   ~ 0
 SPI_MISO
-Text Label 4550 2600 2    50   ~ 0
+Text Label 5000 2400 2    50   ~ 0
 SPI_MOSI
-Text Label 4550 2700 2    50   ~ 0
+Text Label 5000 2200 2    50   ~ 0
 SPI_NSS
 $Comp
@@
 Wire Wire Line
 	6400 2700 6150 2700
-Wire Wire Line
-	3300 2500 3700 2500
 Text Label 5150 1850 0    50   ~ 0
 DIO0
 Wire Wire Line
 	5150 1850 5550 1850
-Text Label 3500 2700 0    50   ~ 0
+Text Label 5000 2100 2    50   ~ 0
 DIO0
 Wire Wire Line
-	3500 2700 3700 2700
+	5000 2200 4650 2200
 Wire Wire Line
-	4550 2700 4200 2700
-Wire Wire Line
-	4200 2600 4550 2600
-Wire Wire Line
-	4550 2500 4200 2500
-Wire Wire Line
-	4200 2400 4550 2400
+	4650 2100 5000 2100
 NoConn ~ 5550 1650
 NoConn ~ 5550 1750
@@
 NoConn ~ 6150 1750
 NoConn ~ 6150 1650
+Wire Wire Line
+	3750 2100 4150 2100
+Wire Wire Line
+	5000 2400 4650 2400
+Wire Wire Line
+	3600 2200 4150 2200
+Wire Wire Line
+	5000 2300 4650 2300
+Wire Wire Line
+	3750 2300 4150 2300
 $EndSCHEMATC
