File: carte_comptage/carte_comptage.kicad_pcb (KiCad board)
At the start: 2 copper layers, 156 parts, among them U1 QRE1113GR, U10 QRE1113GR, U11 QRE1113GR, U12 QRE1113GR, U13 QRE1113GR, U14 QRE1113GR, U15 QRE1113GR, U16 QRE1113GR, U17 QRE1113GR, U18 QRE1113GR, U19 QRE1113GR, U2 QRE1113GR, U20 QRE1113GR, U21 QRE1113GR, U22 QRE1113GR, U23 QRE1113GR, U24 QRE1113GR, U25 QRE1113GR, U26 QRE1113GR, U27 QRE1113GR, U28 QRE1113GR, U29 QRE1113GR, U3 QRE1113GR, U30 QRE1113GR, U31 QRE1113GR, U32 QRE1113GR, U33 AP1117-33, U4 QRE1113GR, U5 QRE1113GR, U6 QRE1113GR, U7 QRE1113GR, U8 QRE1113GR, U9 QRE1113GR

Commit message: debut routage
Parts:
- Dreverse1, Dusb1: value B340 -> B0530W-7-F; footprint Diode_SMD:D_SMC -> B0530W-7-F:SOD3715X145N; moved to B.Cu
- F1: moved to B.Cu
- moved Cbdc3 106.9 mm to (124.5, 128.3)
- moved Jbuck1 106.9 mm to (139.7, 116.8)
- moved Rfb1 106.9 mm to (129.5, 128.3)
- moved Rfb2 106.9 mm to (134.4, 128.3)
- moved Cb1 106.9 mm to (134.6, 118.1)
- moved Cb2 106.9 mm to (130.8, 118.1)
- moved Cbbs1 106.9 mm to (123.2, 120.7)
- moved Cbc1 106.9 mm to (129.5, 123.2)
- moved Cbc2 106.9 mm to (129.5, 125.7)
- moved Cbdc1 106.9 mm to (123.2, 124.5)
- moved Cbdc2 106.9 mm to (125.7, 124.5)
- moved Cbss1 106.9 mm to (120.7, 124.5)
- moved Db1 106.9 mm to (123.2, 118.5)
- moved Lb1 106.9 mm to (131.3, 118.1)
- moved Qor1 106.9 mm to (116.8, 124.5)
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
Commit message: DEBUT ROUTAGE
Parts:
- removed Cb1, Cb2: 47µF, Capacitor_Tantalum_SMD:CP_EIA-6032-28_Kemet-C
- removed Cbbs1, Cdcr1: 100nF, Capacitor_SMD:C_1206_3216Metric
- removed Cbc1: 1nF, Capacitor_SMD:C_1206_3216Metric
- removed Cbc2, Cbss1: 47pF, Capacitor_SMD:C_1206_3216Metric
- removed Cbdc1, Cbdc2: 4.7µF, Capacitor_Tantalum_SMD:CP_EIA-3216-18_Kemet-A
- removed Cbdc3: 10nF, Capacitor_SMD:C_1206_3216Metric
- removed Db1: B340, Diode_SMD:D_SMC
- removed Dreverse1, Dusb1: B0530W-7-F, B0530W-7-F:SOD3715X145N
- removed Jbat1: Conn_01x02, Connector_Phoenix_GMSTB:PhoenixContact_GMSTBA_2,5_2-G-7,62_1x02_P7.62mm_Horizontal
- removed Jbuck1: Conn_01x02, Connector_PinSocket_2.54mm:PinSocket_1x02_P2.54mm_Vertical
- removed Lb1: 6.8µH, Inductor_SMD:L_Wuerth_WE-PD2-Typ-L
- removed Qor1: BSS138, digikey-footprints:SOT-23-3
- removed R41, R42, R43, R44, R49, R50, R51, R52, R57, R58, R59, R60: 15, Resistor_SMD:R_1206_3216Metric
- removed R45, R46, R47, R48, R53, R54, R55, R56, R61, R62, R63, R64: 7.5k, Resistor_SMD:R_1206_3216Metric
- removed Rand1, Rand2: 22k, Resistor_SMD:R_1206_3216Metric
- removed Rbat1: 113k, Resistor_SMD:R_1206_3216Metric
- removed Rbat2, Rfb1: 15k, Resistor_SMD:R_1206_3216Metric
- removed Rbc1: 29.4k, Resistor_SMD:R_1206_3216Metric
- removed Rfb2: 10k, Resistor_SMD:R_1206_3216Metric
- removed buck1: TPS54331D, TPS54331D:SOIC127P599X175-8N
- added Cbdr1: 10µF, Capacitor_Tantalum_SMD:CP_EIA-3216-18_Kemet-A, B.Cu at (90.0, 62.6)
- added Cbdr3: 10µF, Capacitor_Tantalum_SMD:CP_EIA-3216-18_Kemet-A, F.Cu at (179.1, 61.4)
- added Cdcr4: 100nF, Capacitor_SMD:C_1206_3216Metric, F.Cu at (228.3, 44.6)
- added F2: Polyfuse, Resistor_SMD:R_1206_3216Metric, F.Cu at (89.0, 69.0)
- Cdcr2: moved to B.Cu
- F1: moved to F.Cu
- R1, R11, R21, R31, R5: value 15 -> 42
- R12, R13, R14, R15, R2, R22, R23, R24, R25, R3, R32, R33, R34, R35, R4: value 15 -> 7.5k
- R16, R26, R36: value 7.5k -> 42
- moved MUX2 143.7 mm to (195.6, 51.4)
- moved MUX1 116.9 mm to (182.7, 51.4)
- moved Cdcr2 113.4 mm to (88.0, 62.5), turned to 90 degrees
- moved swBoot1 102.3 mm to (206.0, 52.3)
- moved Jtemp1 98.2 mm to (205.6, 45.5), turned to 0 degrees
- moved R5 84.7 mm to (187.8, 111.8)
- moved R38 75.1 mm to (170.9, 111.8)
- moved JxbeeD1 70.1 mm to (93.0, 58.0), turned to 90 degrees
- moved U32 69.9 mm to (170.5, 84.9)
- moved R36 69.9 mm to (193.4, 111.8)
- moved JxbeeG1 69.3 mm to (93.0, 77.0), turned to 90 degrees
- moved U31 65.1 mm to (170.5, 92.2)
- moved R24 64.3 mm to (204.6, 111.2)
- moved U30 63.2 mm to (175.3, 84.9)
- moved R39 62.6 mm to (176.5, 111.8)
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Connections:
- Cdcr2 pad 1: +3V3 -> /V+
- F1 pad 2: +BATT -> VBUS
- R1 pad 1: /Vleds -> /V+
- R10 pad 1: /sheet616FF781/Q28 -> /sheet616FF781/Q7
- R11 pad 1: /Vleds -> /V+
- R12 pad 1: /Vleds -> /sheet616FF781/Q8
- R12 pad 2: Net-(R12-Pad2) -> +3V3
- R13 pad 1: /Vleds -> /sheet616FF781/Q9
- R13 pad 2: Net-(R13-Pad2) -> +3V3
- R14 pad 1: /Vleds -> /sheet616FF781/Q10
- R14 pad 2: Net-(R14-Pad2) -> +3V3
- R15 pad 1: /Vleds -> /sheet616FF781/Q11
- R15 pad 2: Net-(R15-Pad2) -> +3V3
- R16 pad 1: /sheet616FF781/Q1 -> /V+
- R16 pad 2: +3V3 -> Net-(R16-Pad2)
- R17 pad 1: /sheet616FF781/Q8 -> /sheet616FF781/Q12
- R18 pad 1: /sheet616FF781/Q15 -> /sheet616FF781/Q13
- R19 pad 1: /sheet616FF781/Q22 -> /sheet616FF781/Q14
- R2 pad 1: /Vleds -> /sheet616FF781/Q1
- R2 pad 2: Net-(R2-Pad2) -> +3V3
- R20 pad 1: /sheet616FF781/Q29 -> /sheet616FF781/Q15
- R21 pad 1: /Vleds -> /V+
- R22 pad 1: /Vleds -> /sheet616FF781/Q16
- R22 pad 2: Net-(R22-Pad2) -> +3V3
- R23 pad 1: /Vleds -> /sheet616FF781/Q17
- R23 pad 2: Net-(R23-Pad2) -> +3V3
- R24 pad 1: /Vleds -> /sheet616FF781/Q18
- R24 pad 2: Net-(R24-Pad2) -> +3V3
- R25 pad 1: /Vleds -> /sheet616FF781/Q19
- R25 pad 2: Net-(R25-Pad2) -> +3V3
- R26 pad 1: /sheet616FF781/Q2 -> /V+
- R26 pad 2: +3V3 -> Net-(R26-Pad2)
- R27 pad 1: /sheet616FF781/Q9 -> /sheet616FF781/Q20
- R28 pad 1: /sheet616FF781/Q16 -> /sheet616FF781/Q21
- R29 pad 1: /sheet616FF781/Q23 -> /sheet616FF781/Q22
- R3 pad 1: /Vleds -> /sheet616FF781/Q2
- R3 pad 2: Net-(R3-Pad2) -> +3V3
- R30 pad 1: /sheet616FF781/Q30 -> /sheet616FF781/Q23
- R31 pad 1: /Vleds -> /V+
- R32 pad 1: /Vleds -> /sheet616FF781/Q24
- R32 pad 2: Net-(R32-Pad2) -> +3V3
- R33 pad 1: /Vleds -> /sheet616FF781/Q25
- R33 pad 2: Net-(R33-Pad2) -> +3V3
- R34 pad 1: /Vleds -> /sheet616FF781/Q26
- R34 pad 2: Net-(R34-Pad2) -> +3V3
- R35 pad 1: /Vleds -> /sheet616FF781/Q27
- R35 pad 2: Net-(R35-Pad2) -> +3V3
- R36 pad 1: /sheet616FF781/Q3 -> /V+
- R36 pad 2: +3V3 -> Net-(R36-Pad2)
- R37 pad 1: /sheet616FF781/Q10 -> /sheet616FF781/Q28
- R38 pad 1: /sheet616FF781/Q17 -> /sheet616FF781/Q29
- R39 pad 1: /sheet616FF781/Q24 -> /sheet616FF781/Q30
- R4 pad 1: /Vleds -> /sheet616FF781/Q3
- R4 pad 2: Net-(R4-Pad2) -> +3V3
- R5 pad 1: /Vleds -> /V+
- R7 pad 1: /sheet616FF781/Q7 -> /sheet616FF781/Q4
- R8 pad 1: /sheet616FF781/Q14 -> /sheet616FF781/Q5
- R9 pad 1: /sheet616FF781/Q21 -> /sheet616FF781/Q6
- U1 pad 2: GND -> Net-(U1-Pad2)
- U10 pad 1: Net-(R15-Pad2) -> Net-(U10-Pad1)
- U10 pad 2: GND -> Net-(U10-Pad2)
- U10 pad 3: /sheet616FF781/Q29 -> /sheet616FF781/Q9
- U11 pad 1: Net-(R21-Pad2) -> Net-(U10-Pad2)
- U11 pad 2: GND -> Net-(U11-Pad2)
- U11 pad 3: /sheet616FF781/Q2 -> /sheet616FF781/Q10
- U12 pad 1: Net-(R22-Pad2) -> Net-(U11-Pad2)
- U12 pad 3: /sheet616FF781/Q9 -> /sheet616FF781/Q11
- U13 pad 1: Net-(R23-Pad2) -> Net-(R16-Pad2)
- U13 pad 2: GND -> Net-(U13-Pad2)
- U13 pad 3: /sheet616FF781/Q16 -> /sheet616FF781/Q12
- U14 pad 1: Net-(R24-Pad2) -> Net-(U13-Pad2)
- U14 pad 2: GND -> Net-(U14-Pad2)
- U14 pad 3: /sheet616FF781/Q23 -> /sheet616FF781/Q13
- U15 pad 1: Net-(R25-Pad2) -> Net-(U14-Pad2)
- U15 pad 2: GND -> Net-(U15-Pad2)
- U15 pad 3: /sheet616FF781/Q30 -> /sheet616FF781/Q14
- U16 pad 1: Net-(R31-Pad2) -> Net-(U15-Pad2)
- U16 pad 3: /sheet616FF781/Q3 -> /sheet616FF781/Q15
- U17 pad 1: Net-(R32-Pad2) -> Net-(R21-Pad2)
- U17 pad 2: GND -> Net-(U17-Pad2)
- U17 pad 3: /sheet616FF781/Q10 -> /sheet616FF781/Q16
- U18 pad 1: Net-(R33-Pad2) -> Net-(U17-Pad2)
- U18 pad 2: GND -> Net-(U18-Pad2)
- U19 pad 1: Net-(R34-Pad2) -> Net-(U18-Pad2)
- U19 pad 2: GND -> Net-(U19-Pad2)
- U19 pad 3: /sheet616FF781/Q24 -> /sheet616FF781/Q18
- U2 pad 1: Net-(R2-Pad2) -> Net-(U1-Pad2)
- U2 pad 2: GND -> Net-(U2-Pad2)
- U2 pad 3: /sheet616FF781/Q7 -> /sheet616FF781/Q1
- U20 pad 1: Net-(R35-Pad2) -> Net-(U19-Pad2)
- U20 pad 3: /sheet616FF781/Q31 -> /sheet616FF781/Q19
- U21 pad 1: Net-(R41-Pad2) -> Net-(R26-Pad2)
- U21 pad 2: GND -> Net-(U21-Pad2)
- U21 pad 3: /sheet616FF781/Q4 -> /sheet616FF781/Q20
- U22 pad 1: Net-(R42-Pad2) -> Net-(U21-Pad2)
- U22 pad 2: GND -> Net-(U22-Pad2)
- U22 pad 3: /sheet616FF781/Q11 -> /sheet616FF781/Q21
- U23 pad 1: Net-(R43-Pad2) -> Net-(U22-Pad2)
- U23 pad 2: GND -> Net-(U23-Pad2)
- U23 pad 3: /sheet616FF781/Q18 -> /sheet616FF781/Q22
- U24 pad 1: Net-(R44-Pad2) -> Net-(U23-Pad2)
- U24 pad 3: /sheet616FF781/Q25 -> /sheet616FF781/Q23
- U25 pad 1: Net-(R49-Pad2) -> Net-(R31-Pad2)
- U25 pad 2: GND -> Net-(U25-Pad2)
- U25 pad 3: /sheet616FF781/Q5 -> /sheet616FF781/Q24
- U26 pad 1: Net-(R50-Pad2) -> Net-(U25-Pad2)
- U26 pad 2: GND -> Net-(U26-Pad2)
- U26 pad 3: /sheet616FF781/Q12 -> /sheet616FF781/Q25
- U27 pad 1: Net-(R51-Pad2) -> Net-(U26-Pad2)
- U27 pad 2: GND -> Net-(U27-Pad2)
- U27 pad 3: /sheet616FF781/Q19 -> /sheet616FF781/Q26
- U28 pad 1: Net-(R52-Pad2) -> Net-(U27-Pad2)
- U28 pad 3: /sheet616FF781/Q26 -> /sheet616FF781/Q27
- U29 pad 1: Net-(R57-Pad2) -> Net-(R36-Pad2)
- U29 pad 2: GND -> Net-(U29-Pad2)
- U29 pad 3: /sheet616FF781/Q6 -> /sheet616FF781/Q28
- U3 pad 1: Net-(R3-Pad2) -> Net-(U2-Pad2)
- U3 pad 2: GND -> Net-(U3-Pad2)
- U3 pad 3: /sheet616FF781/Q14 -> /sheet616FF781/Q2
- U30 pad 1: Net-(R58-Pad2) -> Net-(U29-Pad2)
- U30 pad 2: GND -> Net-(U30-Pad2)
- U30 pad 3: /sheet616FF781/Q13 -> /sheet616FF781/Q29
- U31 pad 1: Net-(R59-Pad2) -> Net-(U30-Pad2)
- U31 pad 2: GND -> Net-(U31-Pad2)
- U31 pad 3: /sheet616FF781/Q20 -> /sheet616FF781/Q30
- U32 pad 1: Net-(R60-Pad2) -> Net-(U31-Pad2)
- U32 pad 3: /sheet616FF781/Q27 -> /sheet616FF781/Q31
- U4 pad 1: Net-(R4-Pad2) -> Net-(U3-Pad2)
- U4 pad 3: /sheet616FF781/Q21 -> /sheet616FF781/Q3
- U5 pad 2: GND -> Net-(U5-Pad2)
- U5 pad 3: /sheet616FF781/Q28 -> /sheet616FF781/Q4
- U6 pad 1: Net-(R11-Pad2) -> Net-(U5-Pad2)
- U6 pad 2: GND -> Net-(U6-Pad2)
- U6 pad 3: /sheet616FF781/Q1 -> /sheet616FF781/Q5
- U7 pad 1: Net-(R12-Pad2) -> Net-(U6-Pad2)
- U7 pad 2: GND -> Net-(U7-Pad2)
- U7 pad 3: /sheet616FF781/Q8 -> /sheet616FF781/Q6
- U8 pad 1: Net-(R13-Pad2) -> Net-(U7-Pad2)
- U8 pad 3: /sheet616FF781/Q15 -> /sheet616FF781/Q7
- U9 pad 1: Net-(R14-Pad2) -> Net-(R11-Pad2)
- U9 pad 2: GND -> Net-(U10-Pad1)
- U9 pad 3: /sheet616FF781/Q22 -> /sheet616FF781/Q8
- µc1 pad 19: /BAT_SENSE -> Net-(µc1-Pad19)

Commit message: Routage fini, à vérifier, ajouter les encoches de montage
Parts:
- removed Cdcr2, Cdcr4: 100nF, Capacitor_SMD:C_1206_3216Metric
- added Q1: Si2302DS, Package_TO_SOT_SMD:SOT-23, F.Cu at (241.2, 36.2)
- added Ref**: Val**, SVG:drawing, F.Cu at (110.8, 34.2)
- added Rq1: 220, Resistor_SMD:R_1206_3216Metric, F.Cu at (248.8, 41.5)
- added Rq2: 1M, Resistor_SMD:R_1206_3216Metric, F.Cu at (244.2, 36.0)
- Cbdr1: moved to F.Cu
- Cdc1, Clse1, Clse2, Crst1, LSE1, R1, R1w1, Rboot1, Rlse1, Rr1, Rv1, U1, U10, U11, U12, U13, U14, U15, U16, U17, U18, U19, U2, U20, U21, U22, U23, U24, U25, U26, U27, U28, U29, U3, U30, U31, U32, U4, U5, U6, U7, U8, U9: moved to B.Cu
- Jtemp1: footprint Connector_JST:JST_EH_B3B-EH-A_1x03_P2.50mm_Vertical -> Connector_JST:JST_EH_S3B-EH_1x03_P2.50mm_Horizontal
- moved R33 216.9 mm to (2.50, 44.0), turned to 180 degrees
- moved R31 212.5 mm to (12.2, 41.5), turned to 270 degrees
- moved R32 212.3 mm to (2.50, 40.2), turned to 180 degrees
- moved R35 210.9 mm to (16.8, 44.0), turned to 180 degrees
- moved USB1 203.2 mm to (281.8, 35.2), turned to 90 degrees
- moved R34 201.3 mm to (16.8, 40.2), turned to 180 degrees
- moved F1 188.3 mm to (271.2, 23.5), turned to 0 degrees
- moved F2 187.3 mm to (271.2, 25.8), turned to 0 degrees
- moved R37 184.2 mm to (30.2, 40.0), turned to 180 degrees
- moved U33 180.8 mm to (269.0, 31.5), turned to 180 degrees
- moved Cbdr1 180.2 mm to (266.5, 26.5), turned to 180 degrees
- moved U25 179.4 mm to (8.00, 41.0), turned to 90 degrees
- moved U26 173.9 mm to (8.00, 44.8), turned to 90 degrees
- moved R36 168.8 mm to (40.0, 41.2), turned to 270 degrees
- moved JxbeeG1 165.2 mm to (249.2, 23.5)
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Connections:
- F1 pad 1: /V+ -> VBUS
- F1 pad 2: VBUS -> /V+
- F2 pad 1: /V+ -> VBUS
- F2 pad 2: VBUS -> /V+
- JxbeeD1 pad 3: /XBEE_SLEEPING -> /SLEEPING
- JxbeeG1 pad 9: /XBEE_SLEEP -> /SLEEP
- R10 pad 1: /sheet616FF781/Q7 -> /Q7
- R12 pad 1: /sheet616FF781/Q8 -> /Q8
- R13 pad 1: /sheet616FF781/Q9 -> /Q9
- R14 pad 1: /sheet616FF781/Q10 -> /Q10
- R15 pad 1: /sheet616FF781/Q11 -> /Q11
- R17 pad 1: /sheet616FF781/Q12 -> /Q12
- R18 pad 1: /sheet616FF781/Q13 -> /Q13
- R19 pad 1: /sheet616FF781/Q14 -> /Q14
- R2 pad 1: /sheet616FF781/Q1 -> /Q1
- R20 pad 1: /sheet616FF781/Q15 -> /Q15
- R22 pad 1: /sheet616FF781/Q16 -> /Q16
- R23 pad 1: /sheet616FF781/Q17 -> /Q17
- R24 pad 1: /sheet616FF781/Q18 -> /Q18
- R25 pad 1: /sheet616FF781/Q19 -> /Q19
- R27 pad 1: /sheet616FF781/Q20 -> /Q20
- R28 pad 1: /sheet616FF781/Q21 -> /Q21
- R29 pad 1: /sheet616FF781/Q22 -> /Q22
- R3 pad 1: /sheet616FF781/Q2 -> /Q2
- R30 pad 1: /sheet616FF781/Q23 -> /Q23
- R32 pad 1: /sheet616FF781/Q24 -> /Q24
- R33 pad 1: /sheet616FF781/Q25 -> /Q25
- R34 pad 1: /sheet616FF781/Q26 -> /Q26
- R35 pad 1: /sheet616FF781/Q27 -> /Q27
- R37 pad 1: /sheet616FF781/Q28 -> /Q28
- R38 pad 1: /sheet616FF781/Q29 -> /Q29
- R39 pad 1: /sheet616FF781/Q30 -> /Q30
- R4 pad 1: /sheet616FF781/Q3 -> /Q3
- R40 pad 1: /sheet616FF781/Q31 -> /Q31
- R6 pad 1: /sheet616FF781/Q0 -> /Q0
- R7 pad 1: /sheet616FF781/Q4 -> /Q4
- R8 pad 1: /sheet616FF781/Q5 -> /Q5
- R9 pad 1: /sheet616FF781/Q6 -> /Q6
- U1 pad 3: /sheet616FF781/Q0 -> /Q0
- U10 pad 3: /sheet616FF781/Q9 -> /Q9
- U11 pad 3: /sheet616FF781/Q10 -> /Q10
- U12 pad 2: GND -> /sheet616FF781/LED_GND
- U12 pad 3: /sheet616FF781/Q11 -> /Q11
- U13 pad 3: /sheet616FF781/Q12 -> /Q12
- U14 pad 3: /sheet616FF781/Q13 -> /Q13
- U15 pad 3: /sheet616FF781/Q14 -> /Q14
- U16 pad 2: GND -> /sheet616FF781/LED_GND
- U16 pad 3: /sheet616FF781/Q15 -> /Q15
- U17 pad 3: /sheet616FF781/Q16 -> /Q16
- U18 pad 3: /sheet616FF781/Q17 -> /Q17
- U19 pad 3: /sheet616FF781/Q18 -> /Q18
- U2 pad 3: /sheet616FF781/Q1 -> /Q1
- U20 pad 2: GND -> /sheet616FF781/LED_GND
- U20 pad 3: /sheet616FF781/Q19 -> /Q19
- U21 pad 3: /sheet616FF781/Q20 -> /Q20
- U22 pad 3: /sheet616FF781/Q21 -> /Q21
- U23 pad 3: /sheet616FF781/Q22 -> /Q22
- U24 pad 2: GND -> /sheet616FF781/LED_GND
- U24 pad 3: /sheet616FF781/Q23 -> /Q23
- U25 pad 3: /sheet616FF781/Q24 -> /Q24
- U26 pad 3: /sheet616FF781/Q25 -> /Q25
- U27 pad 3: /sheet616FF781/Q26 -> /Q26
- U28 pad 2: GND -> /sheet616FF781/LED_GND
- U28 pad 3: /sheet616FF781/Q27 -> /Q27
- U29 pad 3: /sheet616FF781/Q28 -> /Q28
- U3 pad 3: /sheet616FF781/Q2 -> /Q2
- U30 pad 3: /sheet616FF781/Q29 -> /Q29
- U31 pad 3: /sheet616FF781/Q30 -> /Q30
- U32 pad 2: GND -> /sheet616FF781/LED_GND
- U32 pad 3: /sheet616FF781/Q31 -> /Q31
- U4 pad 2: GND -> /sheet616FF781/LED_GND
- U4 pad 3: /sheet616FF781/Q3 -> /Q3
- U5 pad 3: /sheet616FF781/Q4 -> /Q4
- U6 pad 3: /sheet616FF781/Q5 -> /Q5
- U7 pad 3: /sheet616FF781/Q6 -> /Q6
- U8 pad 2: GND -> /sheet616FF781/LED_GND
- U8 pad 3: /sheet616FF781/Q7 -> /Q7
- U9 pad 3: /sheet616FF781/Q8 -> /Q8
- USB1 pad A6: /USB_D+ -> Net-(USB1-PadA6)
- USB1 pad A7: /USB_D- -> Net-(USB1-PadA7)
- USB1 pad B6: Net-(USB1-PadB6) -> /USB_D+
- USB1 pad B7: Net-(USB1-PadB7) -> /USB_D-
- µc1 pad 10: Net-(µc1-Pad10) -> /S1
- µc1 pad 11: Net-(µc1-Pad11) -> /MUX1
- µc1 pad 14: /LED_R -> /MUX2
- µc1 pad 15: /LED_V -> /LED_EN
- µc1 pad 16: Net-(µc1-Pad16) -> /1W
- µc1 pad 18: Net-(µc1-Pad18) -> /SLEEPING
- µc1 pad 2: Net-(µc1-Pad2) -> /S3
- µc1 pad 20: Net-(µc1-Pad20) -> /LED_R
- µc1 pad 21: Net-(µc1-Pad21) -> /LED_V
- µc1 pad 22: /1W -> Net-(µc1-Pad22)
- µc1 pad 38: /MUX1 -> /SLEEP
- µc1 pad 41: /MUX2 -> Net-(µc1-Pad41)
- µc1 pad 42: /S0 -> Net-(µc1-Pad42)
- µc1 pad 43: /S1 -> Net-(µc1-Pad43)
- µc1 pad 45: /S2 -> Net-(µc1-Pad45)
- µc1 pad 46: /S3 -> Net-(µc1-Pad46)
- µc1 pad 5: Net-(µc1-Pad5) -> /S2
- µc1 pad 6: Net-(µc1-Pad6) -> /S0
Routing:
- net /MUX2: track 0.00 -> 196.2 mm, vias 0 -> 4
- net +3V3: track 0.00 -> 175.9 mm, vias 0 -> 5
- net GND: track 0.00 -> 172.3 mm, vias 0 -> 20
- net /NRST: track 0.00 -> 86.5 mm, vias 0 -> 8
- net /MUX1: track 0.00 -> 82.6 mm, vias 0 -> 2
- net /S2: track 0.00 -> 82.3 mm
- net /V+: track 0.00 -> 80.2 mm, vias 0 -> 1
- net /S3: track 0.00 -> 79.3 mm
- net /S0: track 0.00 -> 68.9 mm
- net /S1: track 0.00 -> 64.3 mm
- net /SWCLK: track 0.00 -> 47.7 mm, vias 0 -> 5
- net /SWDIO: track 0.00 -> 40.8 mm, vias 0 -> 4
- net /BOOT0: track 0.00 -> 36.9 mm, vias 0 -> 2
- net /UART_TX: track 0.00 -> 32.9 mm
- net /UART_RX: track 0.00 -> 31.2 mm
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Other:
- board outline added: 285 x 25 mm

Commit message: Routage fini, à vérifier, ajouter les encoches de montage
Parts:
- JxbeeD1: value Conn_01x10 -> LoRa
- LEDp1: value LED -> POW
- LEDr1: value LED -> LEDR
- LoRa1: value Conn_02x04_Counter_Clockwise -> USB-C
- R1: moved to F.Cu
- SWrst1: value SW_Push -> RST
- moved R31 92.2 mm to (-80.0, 41.5)
- moved R32 92.2 mm to (-89.8, 40.2)
- moved R33 92.2 mm to (-89.8, 44.0)
- moved U25 92.2 mm to (-84.2, 41.0)
- moved U26 92.2 mm to (-84.2, 44.8)
- moved R34 86.5 mm to (-69.8, 40.2)
- moved R35 86.5 mm to (-69.8, 44.0)
- moved U27 86.5 mm to (-64.2, 41.0)
- moved U28 86.5 mm to (-64.2, 44.8)
- moved R36 80.0 mm to (-40.0, 41.5)
- moved R37 80.0 mm to (-49.8, 40.2)
- moved U29 80.0 mm to (-44.2, 41.0)
- moved R38 80.0 mm to (-49.8, 44.0)
- moved U30 80.0 mm to (-44.2, 44.8)
- moved R39 73.5 mm to (-29.8, 40.2)
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Routing:
- net +3V3: track 175.9 -> 813.9 mm, vias 5 -> 30
- net /S1: track 64.3 -> 253.6 mm, vias 0 -> 2
- net /S0: track 68.9 -> 255.0 mm, vias 0 -> 2
- net /S2: track 82.3 -> 247.3 mm
- net /S3: track 79.3 -> 242.5 mm
- net /Q9: track 5.02 -> 125.9 mm
- net /Q8: track 5.52 -> 123.6 mm
- net /Q25: track 5.02 -> 111.3 mm
- net /Q11: track 5.02 -> 108.4 mm
- net /Q24: track 5.02 -> 106.7 mm
- net /Q10: track 5.02 -> 105.6 mm
- net /Q27: track 5.02 -> 91.5 mm
- net /Q13: track 5.02 -> 91.0 mm
- net /Q26: track 5.02 -> 88.7 mm
- net /Q12: track 4.72 -> 87.8 mm
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- added copper zone on F.Cu, net /V+
- added copper zone on B.Cu, net /sheet616FF781/LED_GND
- added copper zone on B.Cu, net GND
- added copper zone on F.Cu, net GND
Other:
- board size 285 x 25 mm -> 378.8 x 25 mm

Commit message: ajouter trous
Parts:
- removed Cbdr3: 10µF, Capacitor_Tantalum_SMD:CP_EIA-3216-18_Kemet-A
- removed Cdc5: 100nF, Capacitor_SMD:C_1206_3216Metric
- removed Cdcp1: 1µF, Capacitor_SMD:C_1206_3216Metric
- removed Ref**: Val**, SVG:drawing
- added C1: 1µF, Capacitor_SMD:C_1206_3216Metric, F.Cu at (260.8, 28.2)
- added C6: 100nF, Capacitor_SMD:C_1206_3216Metric, F.Cu at (262.5, 39.2)
- added Cr2: 10µF, Capacitor_Tantalum_SMD:CP_EIA-3216-18_Kemet-A, F.Cu at (262.8, 28.2)
- Jtemp1: value Conn_01x03 -> 1 WIRE; footprint Connector_JST:JST_EH_S3B-EH_1x03_P2.50mm_Horizontal -> Connector_JST:JST_EH_B3B-EH-A_1x03_P2.50mm_Vertical
- JxbeeD1: value LoRa -> Conn_01x10
- JxbeeG1: value Conn_01x10 -> xBee
- LEDp1: value POW -> LED
- LEDr1: value LEDR -> LED
- LoRa1: value USB-C -> Conn_02x04_Counter_Clockwise
- SWD1: value micromatch -> SWD; footprint 7-215079-6:TE_7-215079-6 -> 7-188275-6:TE_7-188275-6
- SWrst1: value RST -> RESET
- swBoot1: value SW_SPDT -> 0 boot 1
- moved R1w1 31.0 mm to (215.0, 29.8)
- moved Jtemp1 29.2 mm to (216.2, 32.4)
- moved SWD1 3.83 mm to (231.1, 43.0), turned to 90 degrees
- moved LEDp1 2.30 mm to (276.2, 23.2)
- moved LEDr1 1.75 mm to (281.5, 27.2)
- renumbered Cdc1 to C2, Cdc2 to C3, Cdc3 to C4, Cdc4 to C5, Cdc6 to C7, Cdc7 to C8, Cbdr1 to Cr1, Rboot1 to Rb1
Routing:
- net /1W: track 22.0 -> 55.0 mm
- net Net-(USB1-PadS1): track 0.00 -> 19.9 mm
- net GND: track 169.9 -> 163.5 mm, vias 22 -> 28
- net VBUS: track 22.0 -> 28.5 mm
- net /UART_RX: track 31.4 -> 37.5 mm, vias 0 -> 2
- net /SWDIO: track 40.8 -> 45.2 mm
- net /SWCLK: track 47.7 -> 43.7 mm
- net /NRST: track 86.5 -> 82.8 mm
- net Net-(LEDp1-Pad2): track 4.20 -> 2.36 mm
- net +3V3: track 813.9 -> 812.2 mm
- net (no net): track 0.00 -> 1.72 mm
- net /sheet616FF781/LED_GND: track 26.2 -> 27.7 mm
- net Net-(LEDr1-Pad2): track 6.56 -> 7.80 mm
Other:
- board text added: "1"
- board text added: "G-3.3"

Commit message: trous finis, exporter eurocircuit et FreeCAD
Parts:
- added Ref**: Val**, SVG:drawing, F.Cu at (105.2, 35.2)
- Q1, Rq2: moved to B.Cu
- moved Jtemp1 10.1 mm to (226.2, 32.8)
- moved R1w1 10.0 mm to (225.0, 30.2)
- moved Rq2 3.78 mm to (243.8, 32.2), turned to 90 degrees
- moved Q1 3.67 mm to (240.0, 32.8)
- moved Rb1 1.00 mm to (229.5, 28.2)
- moved C8 0.56 mm to (249.8, 34.8)
- moved C3 0.25 mm to (249.8, 30.0)
- moved Cr2 0.25 mm to (263.0, 28.2)
Routing:
- net GND: track 163.5 -> 80.8 mm, vias 28 -> 27
- net /1W: track 55.0 -> 45.5 mm, vias 1 -> 2
- net /SWCLK: track 43.7 -> 50.9 mm, vias 5 -> 6
- net +3V3: track 812.2 -> 806.6 mm
- net Net-(Q1-Pad1): track 15.4 -> 20.3 mm, vias 2 -> 1
- net /S1: track 253.4 -> 257.4 mm, vias 2 -> 4
- net /SWDIO: track 45.2 -> 41.8 mm
- net /V+: track 84.6 -> 81.7 mm
- net /Q25: track 111.3 -> 108.8 mm
- net /sheet616FF781/LED_GND: track 27.7 -> 25.5 mm, vias 1 -> 0
- net /MUX1: track 80.5 -> 78.4 mm
- net /Q29: track 76.2 -> 74.1 mm
- net /S0: track 255.0 -> 253.1 mm
- net /S2: track 247.3 -> 245.5 mm
- net (no net): track 1.72 -> 0.00 mm
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Other:
- board size 378.8 x 25 mm -> 380 x 25 mm
- rule trace_min: 0.2 -> 0

Commit message: carte à vérifier
Routing:
- net /Q7: track 44.0 -> 44.9 mm
- net /Q6: track 36.5 -> 37.4 mm
- net /Q5: track 27.0 -> 27.8 mm
- net /Q18: track 28.9 -> 29.6 mm
- net /Q19: track 32.7 -> 33.3 mm

Commit message: pcb ok
Parts:
- removed JxbeeD1: Conn_01x10, Connector_PinSocket_2.00mm:PinSocket_1x10_P2.00mm_Vertical
- removed JxbeeG1: xBee, Connector_PinSocket_2.00mm:PinSocket_1x10_P2.00mm_Vertical
- removed swBoot1: 0 boot 1, Button_Switch_THT:SW_Slide_1P2T_CK_OS102011MS2Q
- added JXbee1: Conn_02x10_Counter_Clockwise, Xbee:Connector_Xbee, F.Cu at (269.2, 22.3)
- added Jbatt1: Conn_01x02_Male, Connector_JST:JST_EH_B2B-EH-A_1x02_P2.50mm_Vertical, F.Cu at (211.5, 30.3)
- added SwBoot1: RESET, Connector_PinHeader_2.54mm:PinHeader_1x02_P2.54mm_Vertical, F.Cu at (229.0, 24.2)
- LoRa1: footprint Connector_PinHeader_2.54mm:PinHeader_2x04_P2.54mm_Vertical -> Micromatch:ConnectorMicromatch-8
- RledP1: moved to B.Cu
- Rq2: moved to F.Cu
- SWrst1: footprint Button_Switch_SMD:SW_SPST_TL3305C -> Connector_PinSocket_2.54mm:PinSocket_1x02_P2.54mm_Vertical
- moved Rr1 9.66 mm to (283.0, 24.6)
- moved Rv1 9.44 mm to (280.2, 24.6)
- moved Rq1 6.75 mm to (242.0, 41.5)
- moved LoRa1 6.19 mm to (277.7, 42.3), turned to 180 degrees
- moved Rlse1 5.67 mm to (244.8, 30.2), turned to 0 degrees
- moved Rq2 5.46 mm to (245.9, 37.2), turned to -90 degrees
- moved R1w1 4.78 mm to (222.0, 34.0)
- moved SWrst1 4.66 mm to (236.1, 24.2), turned to 90 degrees
- moved LEDv1 3.97 mm to (280.2, 24.6), turned to 90 degrees
- moved LSE1 3.76 mm to (245.8, 32.5)
- moved Jtemp1 3.68 mm to (223.5, 30.3)
- moved RledP1 3.62 mm to (277.5, 24.6)
- moved LEDr1 3.00 mm to (283.0, 24.6), turned to 90 degrees
- moved USB1 2.81 mm to (281.7, 32.4)
- moved C2 2.02 mm to (264.2, 30.2)
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Connections:
- USB1 pad A5: Net-(USB1-PadA5) -> unconnected-(USB1-PadA5)
- USB1 pad A6: Net-(USB1-PadA6) -> unconnected-(USB1-PadA6)
- USB1 pad A7: Net-(USB1-PadA7) -> unconnected-(USB1-PadA7)
- USB1 pad A8: Net-(USB1-PadA8) -> unconnected-(USB1-PadA8)
- USB1 pad B5: Net-(USB1-PadB5) -> unconnected-(USB1-PadB5)
- USB1 pad B8: Net-(USB1-PadB8) -> unconnected-(USB1-PadB8)
- USB1 pad S1: Net-(USB1-PadS1) -> GND
- USB1 pad S2: Net-(USB1-PadS1) -> GND
- USB1 pad S3: Net-(USB1-PadS1) -> GND
- USB1 pad S4: Net-(USB1-PadS1) -> GND
- µc1 pad 17: Net-(µc1-Pad17) -> unconnected-(µc1-Pad17)
- µc1 pad 19: Net-(µc1-Pad19) -> unconnected-(µc1-Pad19)
- µc1 pad 22: Net-(µc1-Pad22) -> unconnected-(µc1-Pad22)
- µc1 pad 30: Net-(µc1-Pad30) -> unconnected-(µc1-Pad30)
- µc1 pad 41: Net-(µc1-Pad41) -> unconnected-(µc1-Pad41)
- µc1 pad 42: Net-(µc1-Pad42) -> unconnected-(µc1-Pad42)
- µc1 pad 43: Net-(µc1-Pad43) -> unconnected-(µc1-Pad43)
- µc1 pad 45: Net-(µc1-Pad45) -> unconnected-(µc1-Pad45)
- µc1 pad 46: Net-(µc1-Pad46) -> unconnected-(µc1-Pad46)
Routing:
- net /V+: track 81.7 -> 452.8 mm
- net /sheet616FF781/LED_GND: track 25.5 -> 318.0 mm
- net VBUS: track 28.5 -> 83.4 mm, vias 0 -> 4
- net Net-(USB1-PadS1): track 19.9 -> 0.00 mm
- net /LED_V: track 22.4 -> 42.1 mm
- net /SLEEPING: track 7.98 -> 26.2 mm, vias 0 -> 3
- net /LED_R: track 27.6 -> 42.1 mm
- net /SLEEP: track 12.2 -> 22.8 mm, vias 0 -> 2
- net /1W: track 45.5 -> 56.1 mm, vias 2 -> 5
- net /SPI_NSS: track 27.6 -> 18.2 mm, vias 0 -> 2
- net /LED_EN: track 8.49 -> 17.8 mm, vias 0 -> 2
- net /MUX1: track 78.4 -> 86.7 mm, vias 0 -> 6
- net /XBEE_DIN: track 9.72 -> 17.7 mm, vias 0 -> 2
- net /DIO0: track 22.5 -> 14.6 mm
- net /SPI_SCK: track 19.1 -> 26.4 mm
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- removed copper zone on F.Cu, net /V+
Other:
- outline, holes or cut-outs redrawn
- net class Default removed
