File: carte_comptage/carte_comptage.kicad_pcb (KiCad board)
At the start: 2 copper layers, 380 x 25 mm, 113 parts, among them Q1 Si2302DS, U1 QRE1113GR, U10 QRE1113GR, U11 QRE1113GR, U12 QRE1113GR, U13 QRE1113GR, U14 QRE1113GR, U15 QRE1113GR, U16 QRE1113GR, U17 QRE1113GR, U18 QRE1113GR, U19 QRE1113GR, U2 QRE1113GR, U20 QRE1113GR, U21 QRE1113GR, U22 QRE1113GR, U23 QRE1113GR, U24 QRE1113GR, U25 QRE1113GR, U26 QRE1113GR, U27 QRE1113GR, U28 QRE1113GR, U29 QRE1113GR, U3 QRE1113GR, U30 QRE1113GR, U31 QRE1113GR, U32 QRE1113GR, U33 AP1117-33, U4 QRE1113GR, U5 QRE1113GR, U6 QRE1113GR, U7 QRE1113GR, U8 QRE1113GR, U9 QRE1113GR

Commit message: ajout jumper coordinateur pcb
Parts:
- added Rb2: 100, Resistor_SMD:R_1206_3216Metric, F.Cu at (266.3, 43.2)
- added SB1: 0, Jumper:SolderJumper-2_P1.3mm_Open_TrianglePad1.0x1.5mm, B.Cu at (275.8, 45.6)
Connections:
- JXbee1 pad 12: unconnected-(JXbee1-Pad12) -> /CTS
- µc1 pad 19: unconnected-(µc1-Pad19) -> /COORD
- µc1 pad 41: unconnected-(µc1-Pad41) -> /CTS
Routing:
- net /CTS: track 0.00 -> 14.1 mm, vias 0 -> 1
- net /COORD: track 0.00 -> 11.1 mm
- net Net-(Rb2-Pad1): track 0.00 -> 7.85 mm, vias 0 -> 1

Commit message: pcb ok
Parts:
- added G***: LOGO, Logo_IUT_Cachan:logo_iut_cachan_SilkScreen, F.Cu at (60.5, 32.1)
- added REF**: KiCad-Logo_5mm_SilkScreen, Symbol:KiCad-Logo_5mm_SilkScreen, F.Cu at (-87.9, 25.9)
- added REF**: ESD-Logo_6.6x6mm_SilkScreen, Symbol:ESD-Logo_6.6x6mm_SilkScreen, F.Cu at (-91.2, 32.5)
- Jbatt1: footprint Connector_JST:JST_EH_B2B-EH-A_1x02_P2.50mm_Vertical -> Connector_JST:JST_PH_B2B-PH-K_1x02_P2.00mm_Vertical
- Jtemp1: footprint Connector_JST:JST_EH_B3B-EH-A_1x03_P2.50mm_Vertical -> Connector_JST:JST_PH_B3B-PH-K_1x03_P2.00mm_Vertical
- Rp1: renamed from RledP1; value 120 -> Rp1
- Rq2: moved to B.Cu
- SB1: moved to F.Cu
- SWrst1: footprint Connector_PinSocket_2.54mm:PinSocket_1x02_P2.54mm_Vertical -> Connector_PinHeader_2.54mm:PinHeader_1x02_P2.54mm_Vertical
- moved SB1 5.69 mm to (270.1, 45.0), turned to -90 degrees
- moved Rb2 4.14 mm to (262.2, 43.0)
- moved Ref** 2.21 mm to (103.1, 35.5)
- moved Jtemp1 1.05 mm to (222.4, 30.3)
- moved R1w1 1.04 mm to (221.0, 34.0)
- moved LoRa1 0.38 mm to (278.1, 42.2)
- moved C4 0.12 mm to (1.25, 25.9)
- moved C5 0.05 mm to (178.5, 25.9)
Routing:
- net /COORD: track 11.1 -> 6.86 mm
- net /V+: track 452.8 -> 449.9 mm
- net +3V3: track 804.3 -> 805.9 mm, vias 35 -> 34
- net /S1: track 256.5 -> 257.6 mm
- net Net-(Rb2-Pad1): track 7.85 -> 6.98 mm, vias 1 -> 0
- net GND: track 76.0 -> 75.9 mm, vias 32 -> 38
Other:
- board text added: "+3V3"
- board text added: "DIO0"
- board text added: "GND"
- board text added: "LoRa"
- board text added: "MUX1 I1 I0"
- board text added: "MUX1 I10 I11"
- board text added: "MUX1 I12 I13"
- board text added: "MUX1 I14 I15"
- board text added: "MUX1 I2 I3"
- board text added: "MUX1 I4 I5"
- board text added: "MUX1 I6 I7"
- board text added: "MUX1 I8 I9"
- board text added: "MUX2 I0 I1"
- board text added: "MUX2 I10 I11"
- board text added: "MUX2 I12 I13"
- board text added: "MUX2 I14 I15"
- board text added: "MUX2 I2 I3"
- board text added: "MUX2 I4 I5"
- board text added: "MUX2 I6 I7"
- board text added: "MUX2 I8 I9"
- board text added: "NRST"
- board text added: "Nicolas Robbe Aslan Halimi Denis Pénard GE1 - S4 - TI"
- board text added: "SB1"
- board text added: "SPI_MISO"
- board text added: "SPI_MOSI"
- board text added: "SPI_NSS"
- board text added: "SPI_SCK"
- board text added: "Solder for COORD >"
- board text removed: "G-3.3"

Commit message: fix
Parts:
- Rp1: value Rp1 -> 120
Connections:
- µc1 pad 31: /BUCK_EN -> unconnected-(µc1-Pad31)
Changed lines of the file:
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@@
   (net 55 "/Q23")
   (net 56 "/MUX2")
-  (net 57 "/BUCK_EN")
+  (net 57 "unconnected-(µc1-Pad31)")
   (net 58 "Net-(R1-Pad2)")
   (net 59 "Net-(R5-Pad2)")
@@
       (net 128 "unconnected-(µc1-Pad30)") (pinfunction "PA9") (pintype "bidirectional+no_connect"))
     (pad "31" smd roundrect locked (at 4.1625 -0.25) (size 1.475 0.3) (layers "F.Cu" "F.Paste" "F.Mask") (roundrect_rratio 0.25)
-      (net 57 "/BUCK_EN") (pinfunction "PA10") (pintype "bidirectional"))
+      (net 57 "unconnected-(µc1-Pad31)") (pinfunction "PA10") (pintype "bidirectional+no_connect"))
     (pad "32" smd roundrect locked (at 4.1625 -0.75) (size 1.475 0.3) (layers "F.Cu" "F.Paste" "F.Mask") (roundrect_rratio 0.25)
       (net 72 "/USB_D-") (pinfunction "PA11") (pintype "bidirectional"))
@@
       (effects (font (size 1 1) (thickness 0.15)) (justify mirror))
     )
-    (fp_text value "Rp1" (at -4 -2.05 90) (layer "B.SilkS")
+    (fp_text value "120" (at -4 -2.05 90) (layer "B.SilkS")
       (effects (font (size 1 1) (thickness 0.15)) (justify mirror))
     )
@@
     (style (thickness 0.15) (arrow_length 1.27) (text_position_mode 0) (extension_height 0.58642) (extension_offset 0) keep_text_aligned)
   )
-  (target plus (at 158.35 29.8) (size 5) (width 0.05) (layer "Edge.Cuts"))
   (target plus (at 65.85 30.7) (size 5) (width 0.05) (layer "Edge.Cuts"))
+  (target plus (at 158.35 29.8) (size 5) (width 0.05) (layer "Edge.Cuts"))
   (segment (start 192.195 26.595) (end 192.195 24.85) (width 0.4) (layer "F.Cu") (net 1))
   (segment (start 281.225 39.65) (end 281.225 37.2725) (width 0.4) (layer "F.Cu") (net 1))

Commit message: carte capteur finie
Parts:
- moved R5 115.5 mm to (295.6, 44.9)
- moved SWD1 115.5 mm to (346.6, 45.6)
- moved SWrst1 115.5 mm to (351.6, 27.2)
- moved C1 115.5 mm to (376.2, 31.2)
- moved C2 115.5 mm to (379.8, 33.2)
- moved C3 115.5 mm to (365.2, 31.5)
- moved C4 115.5 mm to (116.8, 28.9)
- moved C5 115.5 mm to (294.0, 28.9)
- moved C6 115.5 mm to (378.0, 42.2)
- moved C7 115.5 mm to (369.0, 31.0)
- moved C8 115.5 mm to (364.5, 37.8)
- moved Clse1 115.5 mm to (366.2, 31.8)
- moved Clse2 115.5 mm to (363.8, 31.8)
- moved Cr1 115.5 mm to (383.1, 29.5)
- moved Cr2 115.5 mm to (378.5, 31.2)
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
Commit message: fix déplacement silkscreen
Parts:
- moved REF** 159.8 mm to (24.3, 143.1)
- moved G*** 159.8 mm to (176.0, 142.6)
- moved REF** 159.8 mm to (27.6, 136.4)
- moved Ref** 159.8 mm to (218.6, 146.0)
- moved JXbee1 107.5 mm to (384.7, 132.8)
- moved Jbatt1 107.5 mm to (327.0, 140.8)
- moved Jtemp1 107.5 mm to (337.9, 140.8)
- moved Q1 107.5 mm to (355.5, 143.3)
- moved C1 107.5 mm to (376.2, 138.8)
- moved C2 107.5 mm to (379.8, 140.8)
- moved C3 107.5 mm to (365.2, 139.0)
- moved C4 107.5 mm to (116.8, 136.4)
- moved C5 107.5 mm to (294.0, 136.4)
- moved C6 107.5 mm to (378.0, 149.8)
- moved C7 107.5 mm to (369.0, 138.5)
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
Commit message: proto boitier
Routing:
- net +3V3: track 805.9 -> 799.4 mm
- net Net-(Q1-Pad1): track 20.2 -> 15.3 mm
- net /S1: track 257.6 -> 256.5 mm
- net /SLEEP: track 23.3 -> 22.5 mm
- net GND: vias 38 -> 39
