File: carte_comptage/carte_comptage.kicad_sch (KiCad schematic)
At the start: 40 parts, among them Q1 Si2302DS, U33 AP1117-33

Commit message: ajout jumper coordinateur pcb
Parts:
- added Rb2: 100, Resistor_SMD:R_1206_3216Metric, symbol Device:R
- added SB1: 0, Jumper:SolderJumper-2_P1.3mm_Open_TrianglePad1.0x1.5mm, symbol Device:R
Connections:
- net GND: now also SB1.2
- net COORD: now reaches µc1.19 (PB1)
- net COORD: now also Rb2.2
- net CTS: now reaches µc1.41 (PB5)
- net CTS: now also JXbee1.12 (Pin_12)
- new net: Rb2.1, SB1.1
- no-connect marks 29 -> 26
Other:
- note added: "Résistance de 0 ohm : Pont de soudure à faire pour le choix du coord"
- moved on the sheet: Cr1, Cr2, F1, F2, Jbatt1, U33
