File: carte_comptage/carte_comptage.kicad_sch (KiCad schematic)
At the start: 42 parts, among them Q1 Si2302DS, U33 AP1117-33

Commit message: proto boitier
Parts:
- SwBoot1: value RESET -> BOOT
Changed lines of the file:
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@@
       (effects (font (size 1.27 1.27)) (justify right))
     )
-    (property "Value" "RESET" (id 1) (at 260.477 65.9892 90)
+    (property "Value" "BOOT" (id 1) (at 260.477 65.9892 90)
       (effects (font (size 1.27 1.27)) (justify right))
     )
@@
     )
     (path "/27f295c8-a327-467e-9817-2fd5b63dcff9"
-      (reference "SwBoot1") (unit 1) (value "RESET") (footprint "Connector_PinHeader_2.54mm:PinHeader_1x02_P2.54mm_Vertical")
+      (reference "SwBoot1") (unit 1) (value "BOOT") (footprint "Connector_PinHeader_2.54mm:PinHeader_1x02_P2.54mm_Vertical")
     )
     (path "/00000000-0000-0000-0000-0000616ff789/00000000-0000-0000-0000-000061324d32"
