File: carte_comptage/_autosave-carte_comptage.kicad_sch (KiCad schematic)
At the start: 42 parts, among them Q1 Si2302DS, U33 AP1117-33

Commit message: pcb ok
Connections:
- net BUCK_EN: no longer names the net of µc1.31 (PA10)
- no-connect marks 26 -> 27
Changed lines of the file:
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@@
   (no_connect (at 71.12 27.94))
   (no_connect (at 73.66 123.19))
+  (no_connect (at 106.68 128.27))
   (no_connect (at 30.48 35.56))
   (no_connect (at 30.48 27.94))
@@
     (stroke (width 0) (type default) (color 0 0 0 0))
   )
-  (wire (pts (xy 106.68 128.27) (xy 115.57 128.27))
-    (stroke (width 0) (type default) (color 0 0 0 0))
-  )
   (wire (pts (xy 93.98 176.53) (xy 105.41 176.53))
     (stroke (width 0) (type default) (color 0 0 0 0))
@@
     (effects (font (size 1.27 1.27)) (justify left bottom))
   )
-  (label "BUCK_EN" (at 115.57 128.27 180)
-    (effects (font (size 1.27 1.27)) (justify right bottom))
-  )
   (label "USB_D-" (at 80.01 33.02 180)
